File: PonchoEDUCIAA_WIFI_BLT.sch (KiCad schematic (older format))
At the start: 24 parts, among them J1 UART, SW1 Reset, SW2 Boot, U1 ESP32-WROOM

Commit message: Se cambian los leds, sus datasheets y el footprint para unformizar en 0805 smd
Parts:
- D1: footprint LEDs:LED_0402 -> LEDs:LED_0805; Desc LED 5MM 5V VERTICAL RED PC MNT -> LED RED DIFFUSED 0805 SMD; Digikey# 350-1608-ND -> 475-1278-1-ND; Manf Dialight -> OSRAM Opto Semiconductors Inc.; Manf# 5500504F -> LS R976-NR-1; Mouser# 645-550-0504F -> 720-LSR976-NR-1
- D2: footprint LEDs:LED_0402 -> LEDs:LED_0805; Desc LED 5MM VERT HE DIFF GRN PC MNT -> LED GREEN DIFFUSED 0805 SMD; Digikey# 350-2814-ND -> 475-1410-1-ND; Manf Dialight -> OSRAM Opto Semiconductors Inc.; Manf# 5612201050F -> LG R971-KN-1; Mouser# 645-561-2201-050F -> 720-LGR971-KN-1
- D3: footprint LEDs:LED_0402 -> LEDs:LED_0805; Desc LED 5MM 5V VERTICAL YELLOW PCMNT -> LED YELLOW DIFFUSED 0805 SMD; Digikey# 350-1615-ND -> 475-2560-1-ND; Manf Dialight -> OSRAM Opto Semiconductors Inc.; Manf# 5500804F -> LY R976-PS-36; Mouser# 645-550-0804F -> 720-LYR976-PS-36
Changed lines of the file:
@@
 F 0 "D2" V 6400 4200 50  0000 L CNN
 F 1 "LED_Verde" V 6200 4150 50  0000 L CNN
-F 2 "LEDs:LED_0402" V 6300 4150 50  0001 C CNN
-F 3 "http://www.dialight.com/Assets/Brochures_And_Catalogs/Indication/561-xx0x-050.pdf" V 6300 4150 50  0001 C CNN
-F 4 "Dialight" H 6300 4150 60  0001 C CNN "Manf"
-F 5 "5612201050F" H 6300 4150 60  0001 C CNN "Manf#"
-F 6 "350-2814-ND" H 6300 4150 60  0001 C CNN "Digikey#"
-F 7 "645-561-2201-050F" H 6300 4150 60  0001 C CNN "Mouser#"
-F 8 "LED 5MM VERT HE DIFF GRN PC MNT" H 6300 4150 60  0001 C CNN "Desc"
+F 2 "LEDs:LED_0805" V 6300 4150 50  0001 C CNN
+F 3 "http://www.osram-os.com/Graphics/XPic9/00078860_0.pdf" V 6300 4150 50  0001 C CNN
+F 4 "OSRAM Opto Semiconductors Inc." H 6300 4150 60  0001 C CNN "Manf"
+F 5 "LG R971-KN-1" H 6300 4150 60  0001 C CNN "Manf#"
+F 6 "475-1410-1-ND" H 6300 4150 60  0001 C CNN "Digikey#"
+F 7 "720-LGR971-KN-1" H 6300 4150 60  0001 C CNN "Mouser#"
+F 8 "LED GREEN DIFFUSED 0805 SMD" H 6300 4150 60  0001 C CNN "Desc"
 	1    6300 4150
 	0    -1   -1   0
@@
 F 0 "D3" V 6800 4000 50  0000 L CNN
 F 1 "LED_Amarillo" V 6600 3650 50  0000 L CNN
-F 2 "LEDs:LED_0402" V 6700 4150 50  0001 C CNN
-F 3 "http://www.dialight.com/Assets/Brochures_And_Catalogs/Indication/550-xx04.pdf" V 6700 4150 50  0001 C CNN
-F 4 "Dialight" H 6700 4150 60  0001 C CNN "Manf"
-F 5 "5500804F" H 6700 4150 60  0001 C CNN "Manf#"
-F 6 "350-1615-ND" H 6700 4150 60  0001 C CNN "Digikey#"
-F 7 "645-550-0804F" H 6700 4150 60  0001 C CNN "Mouser#"
-F 8 "LED 5MM 5V VERTICAL YELLOW PCMNT" H 6700 4150 60  0001 C CNN "Desc"
+F 2 "LEDs:LED_0805" V 6700 4150 50  0001 C CNN
+F 3 "http://www.osram-os.com/Graphics/XPic9/00078941_0.pdf" V 6700 4150 50  0001 C CNN
+F 4 "OSRAM Opto Semiconductors Inc." H 6700 4150 60  0001 C CNN "Manf"
+F 5 "LY R976-PS-36" H 6700 4150 60  0001 C CNN "Manf#"
+F 6 "475-2560-1-ND" H 6700 4150 60  0001 C CNN "Digikey#"
+F 7 "720-LYR976-PS-36" H 6700 4150 60  0001 C CNN "Mouser#"
+F 8 "LED YELLOW DIFFUSED 0805 SMD" H 6700 4150 60  0001 C CNN "Desc"
 	1    6700 4150
 	0    -1   -1   0
@@
 F 0 "D1" V 7450 5150 50  0000 L CNN
 F 1 "LED_Rojo" V 7400 4650 50  0000 L CNN
-F 2 "LEDs:LED_0402" V 7500 5050 50  0001 C CNN
-F 3 "http://www.dialight.com/Assets/Brochures_And_Catalogs/Indication/550-xx04.pdf" V 7500 5050 50  0001 C CNN
-F 4 "Dialight" H 7500 5050 60  0001 C CNN "Manf"
-F 5 "5500504F" H 7500 5050 60  0001 C CNN "Manf#"
-F 6 "350-1608-ND" H 7500 5050 60  0001 C CNN "Digikey#"
-F 7 "645-550-0504F" H 7500 5050 60  0001 C CNN "Mouser#"
-F 8 "LED 5MM 5V VERTICAL RED PC MNT" H 7500 5050 60  0001 C CNN "Desc"
+F 2 "LEDs:LED_0805" V 7500 5050 50  0001 C CNN
+F 3 "http://www.osram-os.com/Graphics/XPic8/00078896_0.pdf" V 7500 5050 50  0001 C CNN
+F 4 "OSRAM Opto Semiconductors Inc." H 7500 5050 60  0001 C CNN "Manf"
+F 5 "LS R976-NR-1" H 7500 5050 60  0001 C CNN "Manf#"
+F 6 "475-1278-1-ND" H 7500 5050 60  0001 C CNN "Digikey#"
+F 7 "720-LSR976-NR-1" H 7500 5050 60  0001 C CNN "Mouser#"
+F 8 "LED RED DIFFUSED 0805 SMD" H 7500 5050 60  0001 C CNN "Desc"
 	1    7500 5050
 	0    -1   -1   0
